Commit message: git_issue_sorted

File: urdf/zebra.ros2_control.xacro (robot description, xacro)
@@ -1,29 +1,29 @@
 <?xml version="1.0"?>
 <robot xmlns:xacro="http://www.ros.org/wiki/xacro">
-  <!-- Renamed the macro for clarity and added use_sim_time parameter -->
   <xacro:macro name="diffbot_ros2_control" params="name use_sim_time:=false use_mock_hardware:=false prefix:=''">
     <ros2_control name="${name}" type="system">
-      <!-- ***** NEW PART FOR GAZEBO ***** -->
-      <xacro:if value="${use_sim_time}">
-        <hardware>
-          <plugin>gazebo_ros2_control/GazeboSystem</plugin>
-        </hardware>
-      </xacro:if>
       <xacro:unless value="${use_sim_time}">
         <xacro:unless value="${use_mock_hardware}">
           <hardware>
-            <plugin>ros2_control_demo_example_2/DiffBotSystemHardware</plugin>
-            <param name="example_param_hw_start_duration_sec">0</param>
-            <param name="example_param_hw_stop_duration_sec">3.0</param>
+            <plugin>zebra/ZebraSystemHardware</plugin>
+            <param name="loop_rate">30</param>
+            <param name="device">/dev/ttyACM0</param>
+            <param name="baud_rate">115200</param>
+            <param name="timeout_ms">1000</param>
+            <param name="enc_counts_per_rev">2800</param>
           </hardware>
         </xacro:unless>
         <xacro:if value="${use_mock_hardware}">
           <hardware>
-            <plugin>gazebo_ros2_control/GazeboSystem</plugin>
-            <!-- <plugin>mock_components/GenericSystem</plugin>
-            <param name="calculate_dynamics">true</param> -->
+            <plugin>mock_components/GenericSystem</plugin>
+            <param name="calculate_dynamics">true</param>
           </hardware>
         </xacro:if>
       </xacro:unless>
+      <xacro:if value="${use_sim_time}">
+         <hardware>
+          <plugin>gazebo_ros2_control/GazeboSystem</plugin>
+        </hardware>
+      </xacro:if>
       <joint name="${prefix}left_wheel_back_joint">
         <command_interface name="velocity"/>

File: urdf/zebra.urdf.xacro (robot description, xacro)
@@ -1,5 +1,5 @@
 <?xml version="1.0"?>
-<robot name="my_bot" xmlns:xacro="http://www.ros.org/wiki/xacro">
-  <!-- Base link -->
+<robot name="zebra" xmlns:xacro="http://www.ros.org/wiki/xacro">
+	<xacro:include filename="$(find zebra)/urdf/zebra.ros2_control.xacro" />
   <link name="base_link">
     <visual>
@@ -14,14 +14,14 @@
     <inertial>
       <origin xyz="0 0 0.0" rpy="0 0 0"/>
-      <mass value="0.2"/>
-      <inertia ixx="0.01" ixy="0" ixz="0" iyy="0.01" iyz="0" izz="0.02"/>
+      <mass value="2.0"/>
+      <inertia ixx="0.01061" ixy="0" ixz="0" iyy="0.01286" iyz="0" izz="0.0169"/>
     </inertial>
   </link>
   <!-- Gazebo base link properties -->
-  <gazebo reference="base_link">
+  <!-- <gazebo reference="base_link">
     <material>Gazebo/Blue</material>
     <mu1>0.8</mu1>
-    <mu2>0.8</mu2>
-  </gazebo>
+    <mu2>0.1</mu2>
+  </gazebo> -->
   <!-- Wheels -->
   <link name="left_wheel_back">
@@ -37,13 +37,13 @@
     <inertial>
       <origin xyz="0 0 0.0"/>
-      <mass value="0.02"/>
-      <inertia ixx="0.00013" ixy="0" ixz="0" iyy="0.00023" iyz="0" izz="0.00013"/>
-    </inertial>
-  </link>
-  <gazebo reference="left_wheel_back">
+      <mass value="0.2"/>
+      <inertia ixx="0.000167" ixy="0" ixz="0" iyy="0.000167" iyz="0" izz="0.00025"/>
+    </inertial>
+  </link>
+  <!-- <gazebo reference="left_wheel_back">
     <material>Gazebo/Black</material>
-    <mu1>100.0</mu1>
-    <mu2>1000.0</mu2>
-  </gazebo>
+    <mu1>100</mu1>
+    <mu2>1</mu2>
+  </gazebo> -->
   <link name="right_wheel_back">
     <visual>
@@ -58,13 +58,13 @@
     <inertial>
       <origin xyz="0 0 0.0"/>
-      <mass value="0.02"/>
-      <inertia ixx="0.00013" ixy="0" ixz="0" iyy="0.00023" iyz="0" izz="0.00013"/>
-    </inertial>
-  </link>
-  <gazebo reference="right_wheel_back">
+      <mass value="0.2"/>
+      <inertia ixx="0.000167" ixy="0" ixz="0" iyy="0.000167" iyz="0" izz="0.00025"/>
+    </inertial>
+  </link>
+  <!-- <gazebo reference="right_wheel_back">
     <material>Gazebo/Black</material>
-    <mu1>100.0</mu1>
-    <mu2>1000.0</mu2>
-  </gazebo>
+    <mu1>100</mu1>
+    <mu2>1</mu2>
+  </gazebo> -->
   <link name="left_wheel_front">
     <visual>
@@ -79,34 +79,29 @@
     <inertial>
       <origin xyz="0 0 0.0"/>
-      <mass value="0.02"/>
-      <inertia ixx="0.00013" ixy="0" ixz="0" iyy="0.00023" iyz="0" izz="0.00013"/>
-    </inertial>
-  </link>
-  <gazebo reference="left_wheel_front">
+      <mass value="0.2"/>
+      <inertia ixx="0.000167" ixy="0" ixz="0" iyy="0.000167" iyz="0" izz="0.00025"/>
+    </inertial>
+  </link>
+  <link name="right_wheel_front">
+    <visual>
+      <geometry><cylinder length="0.05" radius="0.05"/></geometry>
+      <origin xyz="0 0 0.0" rpy="0 0 0"/>
+      <material name="wheel_black"><color rgba="0.15 0.15 0.15 1.0"/></material>
+    </visual>
+    <collision>
+      <geometry><cylinder length="0.05" radius="0.05"/></geometry>
+      <origin xyz="0 0 0.0" rpy="0 0 0"/>
+    </collision>
+    <inertial>
+      <origin xyz="0 0 0.0"/>
+      <mass value="0.2"/>
+      <inertia ixx="0.000167" ixy="0" ixz="0" iyy="0.000167" iyz="0" izz="0.00025"/>
+    </inertial>
+  </link>
+  <!-- <gazebo reference="right_wheel_front">
     <material>Gazebo/Black</material>
-    <mu1>100.0</mu1>
-    <mu2>1000.0</mu2>
-  </gazebo>
-  <link name="right_wheel_front">
-    <visual>
-      <geometry><cylinder length="0.05" radius="0.05"/></geometry>
-      <origin xyz="0 0 0.0" rpy="0 0 0"/>
-      <material name="wheel_black"><color rgba="0.15 0.15 0.15 1.0"/></material>
-    </visual>
-    <collision>
-      <geometry><cylinder length="0.05" radius="0.05"/></geometry>
-      <origin xyz="0 0 0.0" rpy="0 0 0"/>
-    </collision>
-    <inertial>
-      <origin xyz="0 0 0.0"/>
-      <mass value="0.02"/>
-      <inertia ixx="0.00013" ixy="0" ixz="0" iyy="0.00023" iyz="0" izz="0.00013"/>
-    </inertial>
-  </link>
-  <gazebo reference="right_wheel_front">
-    <material>Gazebo/Black</material>
-    <mu1>10.00</mu1>
-    <mu2>1000.0</mu2>
-  </gazebo>
+    <mu1>100</mu1>
+    <mu2>1</mu2>
+  </gazebo> -->
   <!-- Wheel joints -->
   <joint name="left_wheel_back_joint" type="continuous">
@@ -150,5 +145,5 @@
     <child link="camera_link_optical" />
   </joint>
-  <gazebo reference="camera_link">
+  <!-- <gazebo reference="camera_link">
     <sensor name="rgbd_camera" type="depth">
       <update_rate>30</update_rate>
@@ -175,5 +170,5 @@
       </plugin>
     </sensor>
-  </gazebo>
+  </gazebo> -->
   <!-- <link name="gps_link">
     <sensor name="navsat" type="navsat">
@@ -200,5 +195,5 @@
     </sensor>
   </link> -->
-  <link name ="gps_link">
+  <!-- <link name ="gps_link">
   </link>
   <joint name="gps_joint" type="fixed">
@@ -216,7 +211,7 @@
       </plugin>
     </sensor>
-  </gazebo>
+  </gazebo> -->
     <!-- IMU -->
-  <gazebo reference="base_link">
+  <!-- <gazebo reference="base_link">
     <sensor name="imu_sensor" type="imu">
       <always_on>true</always_on>
@@ -226,5 +221,5 @@
         <frame_name>base_link</frame_name>
       </plugin>
-    </sensor>
+    </sensor> -->
   <!-- GPS -->
     <!-- <sensor name="gps_sensor" type="gps">
@@ -236,6 +231,6 @@
       </plugin>
     </sensor> -->
-  </gazebo>
-  <gazebo>
+  <!-- </gazebo> -->
+  <!-- <gazebo>
     <plugin filename="libgazebo_ros2_control.so" name="gazebo_ros2_control">
       <parameters>$(find my_bot_description)/config/my_bot_controllers.yaml</parameters>
@@ -245,5 +240,5 @@
       </ros>
     </plugin>
-  </gazebo>
+  </gazebo> -->
 <!--
     <xacro:diffbot_ros2_control
@@ -252,3 +247,9 @@
       use_mock_hardware="true" />
   -->
+    <xacro:diffbot_ros2_control
+    name="ZebraSystemHardware"
+    prefix=""
+    use_sim_time="false"
+    use_mock_hardware="false"
+  />
 </robot>
